File: zigbee.cat-toy/hardware/zigbee_toy/zigbee_toy.kicad_sch (KiCad schematic)
At the start: 60 parts, among them J1 USB-C 16P, J2 SWD, J3 LiPo 1S (JST-PH), J4 MOTOR, J5 SPEAKER, Q1 AO3401A, Q2 AO3400A, SW1 PAIR, U1 E73-2G4M08S1C, U2 DRV8213DSGR, U3 LIS2DH12TR, U4 TP4054-42-SOT25R, U5 XB5353A, Y1 32.768k 12.5pF

Commit message: zigbee.cat-toy: rev B board (ESP32-C6), JLC Economic PCBA
- ESP32-C6-MINI-1U-H4 replaces the nRF52840 E73; RT9080 3.3 V regulator,
  1M/1M battery divider, MSKSEMI LIS2DW12TR-MS accelerometer (not ST's),
  one red status LED. Every assembled part is Economic-eligible.
- Module 1 mm from the top edge (JLC Economic edge rule); antenna keepout
  so the PCB-antenna MINI-1 drops onto the same pads.
- Re-routed: USB pair under the module edge, nothing on F.Cu under the
  USB-C, no B.Cu under the crystal, 10 uF at the module 3V3 pin.
- Ball and pod checks cover a MINI-1 antenna overhang.
- README rewritten for rev B; rev A lives under the zigbee.cat-toy/rev-a tag.

Co-Authored-By: Claude Opus 5.5 <noreply@anthropic.com>
Parts:
- removed C7: 100n, Capacitor_SMD:C_0603_1608Metric, symbol Device:C
- removed D3: RED (status), LED_SMD:LED_0603_1608Metric, symbol Device:LED
- removed J2: SWD, Connector_PinHeader_1.27mm:PinHeader_1x05_P1.27mm_Vertical, symbol Connector_Generic:Conn_01x05
- removed R5: 1k, Resistor_SMD:R_0603_1608Metric, symbol Device:R
- removed TP14: INT2, TestPoint:TestPoint_Pad_D1.0mm, symbol Connector:TestPoint
- added C11, C16: 100n, Capacitor_SMD:C_0603_1608Metric, symbol Device:C
- added C5: 1u, Capacitor_SMD:C_0603_1608Metric, symbol Device:C
- added R12, R13: 1M, Resistor_SMD:R_0603_1608Metric, symbol Device:R
- added R14: 68k, Resistor_SMD:R_0603_1608Metric, symbol Device:R
- added R15: 100k, Resistor_SMD:R_0603_1608Metric, symbol Device:R
- added R16, R17: 4.7k, Resistor_SMD:R_0603_1608Metric, symbol Device:R
- added R9: 10k, Resistor_SMD:R_0603_1608Metric, symbol Device:R
- added TP21: EN, TestPoint:TestPoint_Pad_D1.0mm, symbol Connector:TestPoint
- added TP22: GND, TestPoint:TestPoint_Pad_D1.0mm, symbol Connector:TestPoint
- added U6: RT9080-33GJ5, Package_TO_SOT_SMD:TSOT-23-5, symbol zigbee_toy:RT9080
- C8: value 4.7u -> 22u; footprint Capacitor_SMD:C_0603_1608Metric -> Capacitor_SMD:C_0805_2012Metric; LCSC C19666 -> C45783
- C9: value 100n -> 10u; LCSC C14663 -> C19702
- D2: value RED (charging) -> RED (status)
- SW1: value PAIR -> PAIR / BOOT
- TP17: value BTN -> BOOT
- TP2: value VDD -> 3V3
- U1: value E73-2G4M08S1C -> ESP32-C6-MINI-1U-H4; footprint zigbee_toy:Ebyte_E73-2G4M08S1C -> zigbee_toy:ESP32-C6-MINI-1U; symbol zigbee_toy:E73-2G4M08S1C -> zigbee_toy:ESP32-C6-MINI-1U; LCSC C356849 -> C20627095
- U3: value LIS2DH12TR -> LIS2DW12TR-MS; symbol zigbee_toy:LIS2DH12 -> zigbee_toy:LIS2DW12TR-MS; LCSC C110926 -> C50385411
Connections:
- net CHG_LED is gone; now on net LED_A: D2.2 (A), R4.2
- net SWCLK is gone; now on net GND: U1.39 (GND)
- net SWDIO is gone; now on net GND: U1.37 (GND)
- net ACC_INT1: now also U1.16 (IO7), U3.5 (INT1); no longer U1.12 (P0.26), U3.12 (INT1)
- net BTN: now also U1.23 (IO9/BOOT); no longer U1.22 (P0.07)
- net CHG_STAT: now also U1.25 (IO19); no longer D2.1 (K)
- net DBG_TX: now also U1.31 (TXD0/IO16); no longer U1.28 (P0.15)
- net GND: now also D2.1 (K), U1.1 (GND), U1.11 (GND), U1.14 (GND), U1.2 (GND), U1.36 (GND), U1.38 (GND), U1.40 (GND), U1.41 (GND), U1.42 (GND), U1.43 (GND), U1.44 (GND), U1.45 (GND), U1.46 (GND), U1.47 (GND), U1.48 (GND), U1.49 (GND), U1.50 (GND), U1.51 (GND), U1.52 (GND), U1.53 (GND), U3.9 (GND), C11.2, C16.2, C5.2, R13.2, R15.2, TP22.1, U6.2 (GND); no longer U1.21 (GND), U1.24 (GND), U1.5 (GND), U3.5 (Res), U3.6 (GND), U3.7 (GND)
- net I2C_SCL: now also U1.24 (IO18), U3.12 (SCL), R17.2; no longer U1.16 (P0.08), U3.1 (SCL)
- net I2C_SDA: now also U1.22 (IO8), U3.2 (SDA), R16.2; no longer U1.14 (P0.06), U3.4 (SDA)
- net LED_STATUS: now also R4.1, U1.29 (IO23); no longer U1.20 (P0.12)
- net MOT_GAINSEL: now also U1.19 (IO14); no longer U1.4 (P0.28/AIN4)
- net MOT_IPROPI: now also U1.5 (IO2/ADC1_2); no longer U1.3 (P0.03/AIN1)
- net MOT_PWM: now also U1.9 (IO4/ADC1_4); no longer U1.15 (P0.05/AIN3)
- net SPK_PWM: now also U1.10 (IO5/ADC1_5); no longer U1.17 (P1.09)
- net USB_DN: now also U1.17 (IO12/USB_D-); no longer U1.29 (D-)
- net USB_DP: now also U1.18 (IO13/USB_D+); no longer U1.31 (D+)
- net VBAT: now also R12.1, U6.1 (VIN), U6.3 (EN); no longer U1.23 (VDDH)
- net VBUS: now also R14.1; no longer R4.1, U1.27 (VBUS)
- net at U1.32 (NC): now also U1.21 (NC), U1.33 (NC), U1.34 (NC), U1.35 (NC), U1.4 (NC), U1.7 (NC)
- net EN: now reaches U1.8 (EN)
- net EN: now also C5.1, R9.2, TP21.1
- net ACC_INT2: no longer names the net of U3.11 (NC)
- net ACC_INT2: no longer U1.18 (P0.04/AIN2)
- net VDD renamed 3V3
- net 3V3: now also U1.3 (3V3), U3.7 (VDD), C11.1, R16.1, R17.1, R9.1, U6.5 (VOUT); no longer U1.19 (VCC(VDD)), U3.10 (VDD_IO), U3.2 (CS), U3.9 (VDD)
- net XL1 renamed XTAL_P
- net XTAL_P: now also U1.12 (IO0/XTAL_32K_P); no longer U1.11 (XL1/P0.00)
- net XL2 renamed XTAL_N
- net nRESET renamed VBUS_SENSE
- net VBUS_SENSE: now also R14.2, R15.1
- new net VBAT_SENSE: C16.1, R12.2, R13.1, U1.15 (IO6/ADC1_6)
- no-connect marks 20 -> 13
Other:
- note added: "2 uA quiescent, 600 mA, 0.31 V dropout at 600 mA. C8 bulk at the regulator, C9 at module pin 3."
- note added: "3.3 V regulator"
- note added: "Button, status LED, battery sense"
- note added: "D2: GPIO high = on, 1.3 mA. VBAT_SENSE = VBAT / 2, 2.1 uA. C16 holds it for the ADC sample."
- note added: "EN: 10k / 1u power-on delay (Espressif). IO9 = BOOT (SW1). IO8 strap high via R16. IO0/IO1: 32.768 kHz crystal for the light-sleep RTC. IO12/13: USB Serial/JTAG on the charging port. ADC1: IO2 MOT_IPROPI, IO6 VBAT_SENSE. LP (deep-sleep wake): IO7 ACC_INT1."
- note added: "ESP32-C6 module (Zigbee / Thread / BLE / Wi-Fi, USB)"
- note added: "I_chg = 1000 V / R3 = ~300 mA. CHRG (open drain) -> MCU, internal pull-up. VBUS_SENSE = 0.6 x VBUS (3.0 V at 5 V): plugged in, charging or full."
- note added: "MSKSEMI part, not ST: WHO_AM_I 0x11, LIS2DH-style register map. INT2 unused: route wake and tap to INT1. CS and SDO/SA0 open (internal pull-ups): I2C, address 0x19. C10 at VDD, C11 at VDDIO."
- note added: "One board for all three toys (bird / fish / ball). 1S LiPo, protected or not. Battery voltage: VBAT_SENSE (IO6, ADC1_CH6), VBAT / 2. On charger: VBUS_SENSE (IO20). Charging: CHG_STAT (IO19), low = charging. Motor current: MOT_IPROPI (IO2, ADC1_CH2), 0 dB attenuation. GAINSEL: drive low / drive high / input-disconnected = Hi-Z. Motor: DIR (IN1, static) + PWM (IN2): fwd DIR=0 PWM=duty, rev DIR=1 PW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"
- note added: "Test points (back)"
- note added: "USB-C (sink), LiPo charger, USB detect"
- note removed: "Button, status LED, SWD"
- note removed: "C6/C7 at VDDH, C8/C9 at VCC (VDD = REG0 output, 3.0 V via UICR.REGOUT0). REG0 runs as LDO (DCCH unconnected). No 32 kHz crystal inside the module: Y1 is required. PWM nets avoid the low-frequency pins near the radio (P0.02-P0.05, P0.28-P0.31, P1.1x)."
- note removed: "CS = VDD (I2C). SA0 = VDD -> address 0x19. I2C uses the nRF internal pull-ups (~13k, 100 kHz)."
- note removed: "I_chg = 1000 V / R3 = ~300 mA. C4 sits between J1, U4 VCC and U1 VBUS."
- note removed: "One board for all three toys (bird / fish / ball). 1S LiPo, protected or not. Battery voltage: SAADC VDDHDIV5 (internal), no divider. Charging detect: nRF USBDETECTED (VBUS), CHRG drives D2 only. Motor current: SAADC AIN1 (P0.03) on MOT_IPROPI, 0.6 V ref, gain 1. GAINSEL: drive low / drive high / input-disconnected = Hi-Z. Motor: DIR (IN1, static) + PWM (IN2): fwd DIR=0 PWM=duty, rev DIR=1 PWM=1-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"
- note removed: "Test points (back, 1 mm pads, not assembled)"
- note removed: "USB-C (sink) and LiPo charger"
- note removed: "Value = back-silk label. DBG_TX/RX: spare GPIOs, 3 V UART log port (P0.15 / P0.17). PROG: I_chg = V x 300 mA. ISNS: I_motor = V / (A_IPROPI x 1.5k)."
- note removed: "nRF52840 module (Zigbee / BLE / USB)"
- moved on the sheet: C12, C13, C6, C8, C9, D2, R4, TP1, TP10, TP11, TP12, TP13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

Commit message: zigbee.cat-toy: rev B review fixes (driver ground loop, module vias, silk)
From an EE friend's review and the DRV8213 datasheet's layout section:
- C3 flipped so its ground pad drops straight onto the driver's thermal
  pad (return path 14.7 mm -> 1.2 mm); two thermal pad vias instead of one;
  ground via at C2 (18.7 mm -> 4.1 mm)
- IN2 rerouted on the back layer below the driver instead of under it, so
  the back plane under the driver is whole again; EN reshuffled to make room,
  TP21 sits on the EN via
- C2 10 uF -> 22 uF (same part as C1/C8)
- vias in 7 of the module's 9 centre ground pads (module ground to the
  driver 21 mm -> 6.5 mm)
- route generator chamfers 90-degree corners (29 -> 8, the rest inside pads
  or on vias)
- front refs all horizontal, one size; title and paw moved into the bare
  antenna keepout strip on the back
- MOT_DIR/MOT_PWM renamed MOT_IN1/MOT_IN2: PWM drive/brake on both pins
  (drive/coast loses IPROPI while coasting)

Co-Authored-By: Claude Opus 5.5 <noreply@anthropic.com>
Parts:
- C2: value 10u 25V -> 22u; LCSC C15850 -> C45783
- TP7: value PWM -> IN2
- TP8: value DIR -> IN1
Connections:
- net MOT_DIR renamed MOT_IN1
- net MOT_PWM renamed MOT_IN2
Other:
- note added: "One board for all three toys (bird / fish / ball). 1S LiPo, protected or not. Battery voltage: VBAT_SENSE (IO6, ADC1_CH6), VBAT / 2. On charger: VBUS_SENSE (IO20). Charging: CHG_STAT (IO19), low = charging. Motor current: MOT_IPROPI (IO2, ADC1_CH2), 0 dB attenuation. GAINSEL: drive low / drive high / input-disconnected = Hi-Z. Motor PWM = drive/brake: fwd IN1=1, IN2=1-duty; rev IN2=1, IN1=1-duty.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"
- note removed: "One board for all three toys (bird / fish / ball). 1S LiPo, protected or not. Battery voltage: VBAT_SENSE (IO6, ADC1_CH6), VBAT / 2. On charger: VBUS_SENSE (IO20). Charging: CHG_STAT (IO19), low = charging. Motor current: MOT_IPROPI (IO2, ADC1_CH2), 0 dB attenuation. GAINSEL: drive low / drive high / input-disconnected = Hi-Z. Motor: DIR (IN1, static) + PWM (IN2): fwd DIR=0 PWM=duty, rev DIR=1 PW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"
Changed lines of the file:
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@@
 		)
 	)
-	(label "MOT_DIR"
+	(label "MOT_IN1"
 		(at 227.33 110.49 0)
 		(effects
@@
 		)
 	)
-	(label "MOT_PWM"
+	(label "MOT_IN2"
 		(at 227.33 113.03 0)
 		(effects
@@
 		)
 	)
-	(label "MOT_DIR"
+	(label "MOT_IN1"
 		(at 320.04 39.37 180)
 		(effects
@@
 		)
 	)
-	(label "MOT_PWM"
+	(label "MOT_IN2"
 		(at 320.04 41.91 180)
 		(effects
@@
 			)
 		)
-		(property "Value" "10u 25V"
+		(property "Value" "22u"
 			(at 302.26 67.31 0)
 			(effects
@@
 			)
 		)
-		(property "LCSC" "C15850"
+		(property "LCSC" "C45783"
 			(at 299.72 66.04 0)
 			(hide yes)
@@
 			)
 		)
-		(property "Value" "PWM"
+		(property "Value" "IN2"
 			(at 246.38 250.19 90)
 			(effects
@@
 		)
 	)
-	(label "MOT_PWM"
+	(label "MOT_IN2"
 		(at 240.03 248.92 180)
 		(effects
@@
 			)
 		)
-		(property "Value" "DIR"
+		(property "Value" "IN1"
 			(at 246.38 256.54 90)
 			(effects
@@
 		)
 	)
-	(label "MOT_DIR"
+	(label "MOT_IN1"
 		(at 240.03 255.27 180)
 		(effects
@@
 		)
 	)
-	(text "One board for all three toys (bird / fish / ball). 1S LiPo, protected or not.\n\nBattery voltage: VBAT_SENSE (IO6, ADC1_CH6), VBAT / 2.\nOn charger: VBUS_SENSE (IO20). Charging: CHG_STAT (IO19), low = charging.\nMotor current: MOT_IPROPI (IO2, ADC1_CH2), 0 dB attenuation.\nGAINSEL: drive low / drive high / input-disconnected = Hi-Z.\nMotor: DIR (IN1, static) + PWM (IN2): fwd DIR=0 PWM=duty, rev DIR=1 PWM=1-duty.\nMotor: DIR IO3, PWM IO4, GAINSEL IO14.  Speaker: SPK_PWM IO5.  Status LED: LED_STATUS IO23.\n\nTest points: value = back-silk label. TX/RX = UART0, 3.3 V. BOOT low + EN pulse = download mode.\nHand-soldered, not JLC-assembled: J3 battery, J4 motor, J5 speaker.\nAntenna: 2.4 GHz FPC antenna on the module u.FL, plugged in by hand.\nH1, H2: M2 mounting holes (NPTH), diagonal corners; ISO 7380 button head (3.5 mm)."
+	(text "One board for all three toys (bird / fish / ball). 1S LiPo, protected or not.\n\nBattery voltage: VBAT_SENSE (IO6, ADC1_CH6), VBAT / 2.\nOn charger: VBUS_SENSE (IO20). Charging: CHG_STAT (IO19), low = charging.\nMotor current: MOT_IPROPI (IO2, ADC1_CH2), 0 dB attenuation.\nGAINSEL: drive low / drive high / input-disconnected = Hi-Z.\nMotor PWM = drive/brake: fwd IN1=1, IN2=1-duty; rev IN2=1, IN1=1-duty.\nMotor: IN1 IO3, IN2 IO4, GAINSEL IO14.  Speaker: SPK_PWM IO5.  Status LED: LED_STATUS IO23.\n\nTest points: value = back-silk label. TX/RX = UART0, 3.3 V. BOOT low + EN pulse = download mode.\nHand-soldered, not JLC-assembled: J3 battery, J4 motor, J5 speaker.\nAntenna: 2.4 GHz FPC antenna on the module u.FL, plugged in by hand.\nH1, H2: M2 mounting holes (NPTH), diagonal corners; ISO 7380 button head (3.5 mm)."
 		(exclude_from_sim no)
 		(at 15.24 208.28 0)

Commit message: zigbee.cat-toy: rev B shrunk to 36 x 23 mm (was 40 x 26)
- 0402 Basic passives; bulk caps stay 0603/0805. VBUS divider 33k/51k
  (68k has no Basic 0402)
- motor and speaker on JST-SH (SMD, assembled); battery stays JST-PH
- USBLC6-2SC6 on D+/D-; 10 nF on IPROPI (DRV8213 datasheet 8.4.2.2)
- new floorplan and routing: power, driver loop, USB, BTN, the
  accelerometer block and ground vias by hand, the rest Freerouting
  (frozen); every ground pad has its own via or reaches the pour
- module pins 25/26 swapped: VBUS_SENSE on IO19, CHG_STAT on IO20
- the button's two pin-1 pads count as one terminal (KiCad jumper pads)
- gen_silk clips footprint outlines at pads and other parts' silk;
  check_spacing.py checks real body/pad gaps, courtyard overlap is a
  warning
- pod.py and ball.py read the board from placement.py; pod bay grows for
  the 103450 cell; ball board moves so the H2 standoff clears the motor.
  Both --check CLEAN against the new board STEP

Co-Authored-By: Claude Opus 5.5 <noreply@anthropic.com>
Parts:
- added C7: 10n, Capacitor_SMD:C_0402_1005Metric, symbol Device:C
- added U7: USBLC6-2SC6, Package_TO_SOT_SMD:SOT-23-6, symbol Power_Protection:USBLC6-2SC6
- C10, C11, C15, C16, C3: footprint Capacitor_SMD:C_0603_1608Metric -> Capacitor_SMD:C_0402_1005Metric; LCSC C14663 -> C1525
- C12, C13: footprint Capacitor_SMD:C_0603_1608Metric -> Capacitor_SMD:C_0402_1005Metric; LCSC C1648 -> C1554
- C5: footprint Capacitor_SMD:C_0603_1608Metric -> Capacitor_SMD:C_0402_1005Metric; LCSC C15849 -> C52923
- J4: footprint Connector_JST:JST_PH_S2B-PH-K_1x02_P2.00mm_Horizontal -> Connector_JST:JST_SH_SM02B-SRSS-TB_1x02-1MP_P1.00mm_Horizontal; LCSC C173752 -> C160402; Note Side-entry JST-PH, hand-solder (THT) -> Side-entry JST-SH (1 A per pin), SMD; now in the parts list
- J5: footprint Connector_JST:JST_PH_S2B-PH-K_1x02_P2.00mm_Horizontal -> Connector_JST:JST_SH_SM02B-SRSS-TB_1x02-1MP_P1.00mm_Horizontal; LCSC C173752 -> C160402; Note Side-entry JST-PH, hand-solder (THT) -> Side-entry JST-SH, SMD; now in the parts list
- R1, R2: footprint Resistor_SMD:R_0603_1608Metric -> Resistor_SMD:R_0402_1005Metric; LCSC C23186 -> C25905
- R11: footprint Resistor_SMD:R_0603_1608Metric -> Resistor_SMD:R_0402_1005Metric; LCSC C21189 -> C17168
- R12, R13: footprint Resistor_SMD:R_0603_1608Metric -> Resistor_SMD:R_0402_1005Metric; LCSC C22935 -> C26083
- R14: value 68k -> 33k; footprint Resistor_SMD:R_0603_1608Metric -> Resistor_SMD:R_0402_1005Metric; LCSC C23231 -> C25779
- R15: value 100k -> 51k; footprint Resistor_SMD:R_0603_1608Metric -> Resistor_SMD:R_0402_1005Metric; LCSC C25803 -> C25794
- R16, R17: footprint Resistor_SMD:R_0603_1608Metric -> Resistor_SMD:R_0402_1005Metric; LCSC C23162 -> C25900
- R3: footprint Resistor_SMD:R_0603_1608Metric -> Resistor_SMD:R_0402_1005Metric; LCSC C22978 -> C25890
- R4: footprint Resistor_SMD:R_0603_1608Metric -> Resistor_SMD:R_0402_1005Metric; LCSC C21190 -> C11702
- R6: footprint Resistor_SMD:R_0603_1608Metric -> Resistor_SMD:R_0402_1005Metric; LCSC C22843 -> C25867
- R7: footprint Resistor_SMD:R_0603_1608Metric -> Resistor_SMD:R_0402_1005Metric; LCSC C22775 -> C25076
- R8: footprint Resistor_SMD:R_0603_1608Metric -> Resistor_SMD:R_0402_1005Metric; LCSC C25803 -> C25741
- R9: footprint Resistor_SMD:R_0603_1608Metric -> Resistor_SMD:R_0402_1005Metric; LCSC C25804 -> C25744
Connections:
- net CHG_STAT: now also U1.26 (IO20); no longer U1.25 (IO19)
- net GND: now also C7.2, U7.2 (GND)
- net MOT_IPROPI: now also C7.1
- net USB_DN: now also U7.3 (I/O2), U7.4 (I/O2)
- net USB_DP: now also U7.1 (I/O1), U7.6 (I/O1)
- net VBUS: now also U7.5 (VBUS)
- net VBUS_SENSE: now also U1.25 (IO19); no longer U1.26 (IO20)
Other:
- note added: "I_limit = 0.51 V / (R6 x A_IPROPI): GAINSEL low 1.66 A, Hi-Z 324 mA, high 69 mA. C7: IPROPI filter (datasheet 8.4.2.2), 15 us with R6, against motor-cap spikes. Auto-sleep (20 nA) when IN1 = IN2 = 0. Keep the 100 nF cap on the motor tabs."
- note added: "One board for all three toys (bird / fish / ball). 1S LiPo, protected or not. Battery voltage: VBAT_SENSE (IO6, ADC1_CH6), VBAT / 2. On charger: VBUS_SENSE (IO19). Charging: CHG_STAT (IO20), low = charging. Motor current: MOT_IPROPI (IO2, ADC1_CH2), 0 dB attenuation. GAINSEL: drive low / drive high / input-disconnected = Hi-Z. Motor PWM = drive/brake: fwd IN1=1, IN2=1-duty; rev IN2=1, IN1=1-duty.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"
- note removed: "I_limit = 0.51 V / (R6 x A_IPROPI): GAINSEL low 1.66 A, Hi-Z 324 mA, high 69 mA. Auto-sleep (20 nA) when IN1 = IN2 = 0. Keep the 100 nF cap on the motor tabs."
- note removed: "One board for all three toys (bird / fish / ball). 1S LiPo, protected or not. Battery voltage: VBAT_SENSE (IO6, ADC1_CH6), VBAT / 2. On charger: VBUS_SENSE (IO20). Charging: CHG_STAT (IO19), low = charging. Motor current: MOT_IPROPI (IO2, ADC1_CH2), 0 dB attenuation. GAINSEL: drive low / drive high / input-disconnected = Hi-Z. Motor PWM = drive/brake: fwd IN1=1, IN2=1-duty; rev IN2=1, IN1=1-duty.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"
