File: zigbee.cat-toy/hardware/zigbee_toy/zigbee_toy.kicad_sch (KiCad schematic)
At the start: 70 parts, among them J1 USB-C 16P, J3 LiPo 1S (JST-PH), J4 MOTOR, J5 SPEAKER, Q1 AO3401A, Q2 AO3400A, SW1 PAIR / BOOT, U1 ESP32-C6-MINI-1U-H4, U2 DRV8213DSGR, U3 LIS2DW12TR-MS, U4 TP4054-42-SOT25R, U5 XB5353A, U6 RT9080-33GJ5, U7 USBLC6-2SC6, Y1 32.768k 12.5pF

Commit message: zigbee.cat-toy: fixes from the rev B datasheet review
docs/design_review_rev_b.md (Fable) found three must-fix issues:
- USBLC6 pin 5 moves from VBUS to 3V3: the C6 enables its D+ pull-up
  from boot, which back-fed VBUS through the steering diode while
  unplugged (~1.7 V on VBUS_SENSE, ~75 uA leak through the divider and
  the TP4054). U7 rotated so pin 5 faces the module side; BTN rerouted on
  the back along the top and down the right edge to free that corridor
- R10 10k pull-up on CHG_STAT: the TP4054's charge-done state is a
  20 uA pull-down, which beats the C6's internal ~45k pull-up
- charge current is 260 mA with R3 = 3.3k (1000/I only holds to
  150 mA); docs corrected, R3 kept (cooler charger)

README: firmware notes from the review (low-battery cutoff, charge-state
decode, driver auto-sleep, 324 mA default for the JST-SH motor lead,
charger heat) and the review's should-fix items listed as open.
DRC clean, spacing ok, JLC export 47 parts, pod/ball --check CLEAN.

Co-Authored-By: Claude Opus 5.5 <noreply@anthropic.com>
Parts:
- added R10: 10k, Resistor_SMD:R_0402_1005Metric, symbol Device:R
Connections:
- net 3V3: now also U7.5 (VBUS), R10.1
- net CHG_STAT: now also R10.2
- net USB_DN: now also U7.1 (I/O1), U7.6 (I/O1); no longer U7.3 (I/O2), U7.4 (I/O2)
- net USB_DP: now also U7.3 (I/O2), U7.4 (I/O2); no longer U7.1 (I/O1), U7.6 (I/O1)
- net VBUS: no longer U7.5 (VBUS)
Other:
- note added: "I_chg = (1000 V / R3) x (1.2 - 4 I/3) = 260 mA. CHRG -> MCU, R10 pull-up (its done-state pull-down is weak). U7 pin 5 on 3V3, not VBUS: the C6 pulls D+ up while unplugged and would back-feed VBUS. VBUS_SENSE = 0.61 x VBUS (3.0 V at 5 V): plugged in, charging or full."
- note removed: "I_chg = 1000 V / R3 = ~300 mA. CHRG (open drain) -> MCU, internal pull-up. VBUS_SENSE = 0.6 x VBUS (3.0 V at 5 V): plugged in, charging or full."
- moved on the sheet: U7
Changed lines of the file:
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@@
 	(symbol
 		(lib_id "Power_Protection:USBLC6-2SC6")
-		(at 68.58 118.11 0)
+		(at 58.42 118.11 0)
 		(unit 1)
 		(exclude_from_sim no)
@@
 		(dnp no)
 		(property "Reference" "U7"
-			(at 69.215 112.395 0)
+			(at 59.055 112.395 0)
 			(effects
 				(font
@@
 		)
 		(property "Value" "USBLC6-2SC6"
-			(at 69.215 114.3 0)
+			(at 59.055 114.3 0)
 			(effects
 				(font
@@
 		)
 		(property "Footprint" "Package_TO_SOT_SMD:SOT-23-6"
-			(at 69.85 124.46 0)
+			(at 59.69 124.46 0)
 			(hide yes)
 			(effects
@@
 		)
 		(property "LCSC" "C7519"
-			(at 68.58 118.11 0)
+			(at 58.42 118.11 0)
 			(hide yes)
 			(effects
@@
 		)
 		(property "Datasheet" "https://www.st.com/resource/en/datasheet/usblc6-2.pdf"
-			(at 69.85 126.365 0)
+			(at 59.69 126.365 0)
 			(hide yes)
 			(effects
@@
 		)
 		(property "Description" "Very low capacitance ESD protection diode, 2 data-line, SOT-23-6"
-			(at 68.58 118.11 0)
+			(at 58.42 118.11 0)
 			(hide yes)
 			(effects
@@
 	(wire
 		(pts
-			(xy 63.5 118.11)
-			(xy 60.96 118.11)
-		)
-		(stroke
-			(width 0)
-			(type default)
-		)
-	)
-	(label "USB_DP"
-		(at 60.96 118.11 180)
+			(xy 53.34 118.11)
+			(xy 50.8 118.11)
+		)
+		(stroke
+			(width 0)
+			(type default)
+		)
+	)
+	(label "USB_DN"
+		(at 50.8 118.11 180)
 		(effects
 			(font
@@
 	(wire
 		(pts
-			(xy 68.58 125.73)
-			(xy 68.58 128.27)
+			(xy 58.42 125.73)
+			(xy 58.42 128.27)
 		)
 		(stroke
@@
 	(symbol
 		(lib_id "power:GND")
-		(at 68.58 128.27 0)
+		(at 58.42 128.27 0)
 		(unit 1)
 		(exclude_from_sim no)
@@
 		(dnp no)
 		(property "Reference" "#PWR07"
-			(at 68.58 134.62 0)
+			(at 58.42 134.62 0)
 			(hide yes)
 			(effects
@@
 		)
 		(property "Value" "GND"
-			(at 68.58 132.08 0)
+			(at 58.42 132.08 0)
 			(effects
 				(font
@@
 		)
 		(property "Footprint" ""
-			(at 68.58 128.27 0)
+			(at 58.42 128.27 0)
 			(hide yes)
 			(effects
@@
 		)
 		(property "Datasheet" ""
-			(at 68.58 128.27 0)
+			(at 58.42 128.27 0)
 			(hide yes)
 			(effects
@@
 		)
 		(property "Description" "Power symbol creates a global label with name \"GND\" , ground"
-			(at 68.58 128.27 0)
+			(at 58.42 128.27 0)
 			(hide yes)
 			(effects
@@
 	(wire
 		(pts
+			(xy 53.34 120.65)
+			(xy 50.8 120.65)
+		)
+		(stroke
+			(width 0)
+			(type default)
+		)
+	)
+	(label "USB_DP"
+		(at 50.8 120.65 180)
+		(effects
+			(font
+				(size 1.27 1.27)
+			)
+			(justify right bottom)
+		)
+	)
+	(wire
+		(pts
 			(xy 63.5 120.65)
-			(xy 60.96 120.65)
+			(xy 66.04 120.65)
+		)
+		(stroke
+			(width 0)
+			(type default)
+		)
+	)
+	(label "USB_DP"
+		(at 66.04 120.65 0)
+		(effects
+			(font
+				(size 1.27 1.27)
+			)
+			(justify left bottom)
+		)
+	)
+	(wire
+		(pts
+			(xy 58.42 113.03)
+			(xy 58.42 110.49)
+		)
+		(stroke
+			(width 0)
+			(type default)
+		)
+	)
+	(label "3V3"
+		(at 58.42 110.49 90)
+		(effects
+			(font
+				(size 1.27 1.27)
+			)
+			(justify left bottom)
+		)
+	)
+	(wire
+		(pts
+			(xy 63.5 118.11)
+			(xy 66.04 118.11)
 		)
 		(stroke
@@
 	)
 	(label "USB_DN"
-		(at 60.96 120.65 180)
-		(effects
-			(font
-				(size 1.27 1.27)
-			)
-			(justify right bottom)
-		)
-	)
-	(wire
-		(pts
-			(xy 73.66 120.65)
-			(xy 76.2 120.65)
-		)
-		(stroke
-			(width 0)
-			(type default)
-		)
-	)
-	(label "USB_DN"
-		(at 76.2 120.65 0)
-		(effects
-			(font
-				(size 1.27 1.27)
-			)
-			(justify left bottom)
-		)
-	)
-	(wire
-		(pts
-			(xy 68.58 113.03)
-			(xy 68.58 110.49)
-		)
-		(stroke
-			(width 0)
-			(type default)
-		)
-	)
-	(label "VBUS"
-		(at 68.58 110.49 90)
-		(effects
-			(font
-				(size 1.27 1.27)
-			)
-			(justify left bottom)
-		)
-	)
-	(wire
-		(pts
-			(xy 73.66 118.11)
-			(xy 76.2 118.11)
-		)
-		(stroke
-			(width 0)
-			(type default)
-		)
-	)
-	(label "USB_DP"
-		(at 76.2 118.11 0)
+		(at 66.04 118.11 0)
 		(effects
 			(font
@@
 	)
 	(symbol
+		(lib_id "Device:R")
+		(at 86.36 144.78 0)
+		(unit 1)
+		(exclude_from_sim no)
+		(in_bom yes)
+		(on_board yes)
+		(dnp no)
+		(property "Reference" "R10"
+			(at 88.9 143.51 0)
+			(effects
+				(font
+					(size 1.27 1.27)
+				)
+				(justify left)
+			)
+		)
+		(property "Value" "10k"
+			(at 88.9 146.05 0)
+			(effects
+				(font
+					(size 1.27 1.27)
+				)
+				(justify left)
+			)
+		)
+		(property "Footprint" "Resistor_SMD:R_0402_1005Metric"
+			(at 84.582 144.78 0)
+			(hide yes)
+			(effects
+				(font
+					(size 1.27 1.27)
+				)
+			)
+		)
+		(property "LCSC" "C25744"
+			(at 86.36 144.78 0)
+			(hide yes)
+			(effects
+				(font
+					(size 1.27 1.27)
+				)
+			)
+		)
+		(property "Datasheet" ""
+			(at 86.36 144.78 0)
+			(hide yes)
+			(effects
+				(font
+					(size 1.27 1.27)
+				)
+			)
+		)
+		(property "Description" "Resistor"
+			(at 86.36 144.78 0)
+			(hide yes)
+			(effects
+				(font
+					(size 1.27 1.27)
+				)
+			)
+		)
+		(pin "1"
+		)
+		(pin "2"
+		)
+		(instances
+			(project "zigbee_toy"
+				(path "/cd6f7973-3019-533d-a0cf-98d98a659f5e"
+					(reference "R10")
+					(unit 1)
+				)
+			)
+		)
+	)
+	(wire
+		(pts
+			(xy 86.36 140.97)
+			(xy 86.36 138.43)
+		)
+		(stroke
+			(width 0)
+			(type default)
+		)
+	)
+	(label "3V3"
+		(at 86.36 138.43 90)
+		(effects
+			(font
+				(size 1.27 1.27)
+			)
+			(justify left bottom)
+		)
+	)
+	(wire
+		(pts
+			(xy 86.36 148.59)
+			(xy 86.36 151.13)
+		)
+		(stroke
+			(width 0)
+			(type default)
+		)
+	)
+	(label "CHG_STAT"
+		(at 86.36 151.13 270)
+		(effects
+			(font
+				(size 1.27 1.27)
+			)
+			(justify right bottom)
+		)
+	)
+	(symbol
 		(lib_id "Device:C")
 		(at 93.98 171.45 0)
@@
 		)
 	)
-	(text "I_chg = 1000 V / R3 = ~300 mA.  CHRG (open drain) -> MCU, internal pull-up.\nVBUS_SENSE = 0.6 x VBUS (3.0 V at 5 V): plugged in, charging or full."
+	(text "I_chg = (1000 V / R3) x (1.2 - 4 I/3) = 260 mA.  CHRG -> MCU, R10 pull-up (its done-state pull-down is weak).\nU7 pin 5 on 3V3, not VBUS: the C6 pulls D+ up while unplugged and would back-feed VBUS.\nVBUS_SENSE = 0.61 x VBUS (3.0 V at 5 V): plugged in, charging or full."
 		(exclude_from_sim no)
 		(at 15.24 184.15 0)

Commit message: zigbee.cat-toy: rev B review should-fix items
- C14 100 nF at module pin 3, beside C9. C2 moves 0.45 mm west to make
  room; the router's GAINSEL detour along the top edge is gone.
- R5 10 k pull-up on IO9 (BOOT). Its BTN via runs on the back to TP17,
  just below the antenna keepout; GAINSEL drops to a lane under it and
  TP21 (EN) moves down the EN route.
- Accelerometer pad 4 to GND, per the datasheet's connection column.
  ACC_INT1 now crosses under the sensor; TP13 moves onto its vertical.
- Two ground vias under the TP4054 on pin 2. The VBAT lane dips below
  them; TP20 and TP22 move off the charger's underside.
- gen_silk drops a pin-1 dot that lands on a neighbour's pad.

Co-Authored-By: Claude Opus 5.5 <noreply@anthropic.com>
Parts:
- added C14: 100n, Capacitor_SMD:C_0402_1005Metric, symbol Device:C
- added R5: 10k, Resistor_SMD:R_0402_1005Metric, symbol Device:R
Connections:
- net 3V3: now also C14.1, R5.1
- net BTN: now also R5.2
- net GND: now also U3.4 (NC), C14.2
- no-connect marks 13 -> 12
Other:
- note added: "2 uA quiescent, 600 mA, 0.31 V dropout at 600 mA. C8 bulk at the regulator, C9 + C14 at module pin 3."
- note added: "D2: GPIO high = on, 1.3 mA. R5: IO9 (BOOT strap) pull-up, per the C6 design guidelines. VBAT_SENSE = VBAT / 2, 2.1 uA. C16 holds it for the ADC sample."
- note added: "MSKSEMI part, not ST: WHO_AM_I 0x11, LIS2DH-style register map. INT2 unused: route wake and tap to INT1. CS and SDO/SA0 open (internal pull-ups): I2C, address 0x19. C10 at VDD, C11 at VDDIO. Pin 4: NC in the pin table, GND in its connection column for every mode, so grounded."
- note removed: "2 uA quiescent, 600 mA, 0.31 V dropout at 600 mA. C8 bulk at the regulator, C9 at module pin 3."
- note removed: "D2: GPIO high = on, 1.3 mA. VBAT_SENSE = VBAT / 2, 2.1 uA. C16 holds it for the ADC sample."
- note removed: "MSKSEMI part, not ST: WHO_AM_I 0x11, LIS2DH-style register map. INT2 unused: route wake and tap to INT1. CS and SDO/SA0 open (internal pull-ups): I2C, address 0x19. C10 at VDD, C11 at VDDIO."
